Commit message: Stuff an tings

File: vrx_urdf/wamv_gazebo/urdf/components/wamv_imu.xacro (robot description, xacro)
@@ -1,5 +1,5 @@
 <?xml version="1.0"?>
 <robot xmlns:xacro="http://ros.org/wiki/xacro">
-  <xacro:macro name="wamv_imu" params="name:=imu x:=0.3 y:=0.5 z:=1.3 R:=0 P:=0 Y:=0 update_rate:=100">
+  <xacro:macro name="wamv_imu" params="name:=imu x:=0.3 y:=0.5 z:=1.3 R:=0 P:=0 Y:=0 update_rate:=10">
     <link name="${namespace}/${name}_link">
       <visual name="${name}_visual">>
@@ -32,5 +32,5 @@
         <update_rate>${update_rate}</update_rate>
         <imu>
-          <angular_velocity>
+          <!-- <angular_velocity>
             <x>
               <noise type="gaussian">
@@ -101,5 +101,5 @@
               </noise>
             </z>
-          </linear_acceleration>
+          </linear_acceleration> -->
           <orientation_reference_frame>
             <localization>ENU</localization>

File: vrx_urdf/wamv_gazebo/urdf/wamv_gazebo.urdf.xacro (robot description, xacro)
@@ -89,4 +89,12 @@
       name="gz::sim::systems::JointStatePublisher">
     </plugin>
+    <plugin
+      filename="gz-sim-odometry-publisher-system"
+      name="gz::sim::systems::OdometryPublisher">
+      <odom_frame>$(arg namespace)/odometry</odom_frame>
+      <robot_base_frame>$(arg namespace)</robot_base_frame>
+      <dimensions>3</dimensions>
+      <odom_publish_frequency>20</odom_publish_frequency>
+    </plugin>
   </gazebo>
   <!-- === Sensors === -->
@@ -115,5 +123,5 @@
     <!-- Add 3D LIDAR -->
     <xacro:if value="$(arg lidar_enabled)">
-      <xacro:lidar name="lidar_wamv" y="-0.3" type="16_beam"/>
+      <xacro:lidar name="lidar_wamv" y="-0.3" type="32_beam"/>
     </xacro:if>
     <!-- Add P3D ground truth -->
@@ -135,8 +143,8 @@
       <xacro:cpu_cases position="-0.15 0 1.53" orientation="0 0 0"/>
       <!-- Add a stereo camera pair -->
-      <xacro:wamv_camera name="front_left_camera" y="0.1" x="0.75" P="${radians(15)}" />
-      <xacro:wamv_camera name="front_right_camera" y="-0.1" x="0.75" P="${radians(15)}" />
+      <!-- <xacro:wamv_camera name="front_left_camera" y="0.1" x="0.75" P="${radians(15)}" />
+      <xacro:wamv_camera name="front_right_camera" y="-0.1" x="0.75" P="${radians(15)}" /> -->
       <!-- Add a camera facing right -->
-      <xacro:wamv_camera name="middle_right_camera" y="-0.45" P="${radians(15)}" Y="${radians(-90)}" post_Y="${radians(-90)}" />
+      <!-- <xacro:wamv_camera name="middle_right_camera" y="-0.45" P="${radians(15)}" Y="${radians(-90)}" post_Y="${radians(-90)}" /> -->
       <!-- Add simulated GPS -->
       <xacro:wamv_gps name="gps_wamv" x="-0.85" />
@@ -144,9 +152,9 @@
       <xacro:wamv_imu name="imu_wamv" y="-0.2" />
       <!-- Add 3D LIDAR -->
-      <xacro:lidar name="lidar_wamv" type="16_beam"/>
+      <xacro:lidar name="lidar_wamv" x="0.43" z="1.93" type="32_beam"/>
       <!-- Add pinger -->
-      <xacro:wamv_pinger sensor_name="receiver" position="-528 191 -2.0" />
+      <!-- <xacro:wamv_pinger sensor_name="receiver" position="-528 191 -2.0" /> -->
       <!-- Add ball shooter (default pitch angle: ~-60 deg) -->
-      <xacro:wamv_ball_shooter name="ball_shooter" x="0.54" y="0.30" z="1.296" pitch="-1.04"/>
+      <!-- <xacro:wamv_ball_shooter name="ball_shooter" x="0.54" y="0.30" z="1.296" pitch="-1.04"/> -->
     </xacro:if>
   </xacro:unless>
